File: Contra.sch (KiCad schematic (older format))
At the start: 103 parts, among them P1 Pad, P2 Pad, P3 Pad, P4 Pad, SW1 SW_PUSH, U1 ProMicro

Commit message: initial commit for wireless mods for BlueMicro
Parts:
- removed P1, P2, P3, P4: Pad, locallib:mountinghole, symbol R
- added J1, J2, J3, J4, J5, J6, J7, J8: Conn_01x01, MountingHole:MountingHole_2.2mm_M2_ISO7380, symbol Connector_Generic:Conn_01x01
- added J10: Conn_01x02, Connector_PinHeader_2.54mm:PinHeader_1x02_P2.54mm_Vertical, symbol Connector_Generic:Conn_01x02
- added J9: Conn_01x04, Connector_PinHeader_2.54mm:PinHeader_1x04_P2.54mm_Vertical, symbol Connector_Generic:Conn_01x04
- added SW2: SW_SPDT, footprints:SPDT_C128955, symbol Switch:SW_SPDT
- D1, D10, D11, D12, D13, D14, D15, D16, D17, D18, D19, D2, D20, D21, D22, D23, D24, D25, D26, D27, D28, D29, D3, D30, D31, D32, D33, D34, D35, D36, D37, D38, D39, D4, D40, D41, D42, D43, D44, D45, D46, D47, D48, D5, D6, D7, D8, D9: footprint Diodes_THT:D_DO-35_SOD27_P7.62mm_Horizontal -> footprints:D_SOD123_axial-dual; symbol D_Small -> Device:D_Small
- MX1, MX10, MX11, MX12, MX13, MX14, MX15, MX16, MX17, MX18, MX19, MX2, MX20, MX21, MX22, MX23, MX24, MX25, MX26, MX27, MX28, MX29, MX3, MX30, MX31, MX32, MX33, MX34, MX35, MX36, MX37, MX38, MX39, MX4, MX40, MX41, MX42, MX43, MX44, MX45, MX46, MX47, MX48, MX5, MX6, MX7, MX8, MX9: symbol MX-1U -> Contra-rescue:MX-1U
- MX49: symbol MX-2U -> Contra-rescue:MX-2U
- SW1: footprint Molex-0548190589:PushButton_6x6mm_TH -> footprints:SW_TACT_ALPS_SKQGABE010; symbol SW_PUSH -> Contra-rescue:SW_PUSH
- U1: symbol ProMicro -> josh:ProMicro
Connections:
- wire segments 70 -> 162
- no-connect marks 0 -> 1
Other:
- moved on the sheet: SW1
